File: Internal_40KB/KiCad/VIC-20_Internal_40KB_RAM.kicad_pcb (KiCad board)
At the start: 2 copper layers, 66 x 62.2 mm, 18 parts, among them J1 BLK Decoder, J2 RAM Decoder, J3 Disable/Enable Switch, J4 UD4, J5 UE4, U1 74LS20, U2 74LS138, U3 74LS138, U4 74HCT30, U5 74LS157, U6 CY62128Exx-xxS

Commit message: Initial design completed
Parts:
- moved C5 0.76 mm to (92.9, 79.8), turned to 180 degrees
- moved U4 0.30 mm to (88.8, 56.0)
- moved U2 0.20 mm to (88.6, 71.1)
Routing:
- net +5V: track 0.00 -> 298.7 mm, vias 0 -> 2
- net /VA11: track 0.00 -> 88.1 mm, vias 0 -> 2
- net /CA15: track 0.00 -> 85.0 mm, vias 0 -> 2
- net /VA10: track 0.00 -> 78.3 mm
- net /CA14: track 0.00 -> 77.2 mm, vias 0 -> 2
- net /CA13: track 0.00 -> 75.3 mm, vias 0 -> 4
- net /~{RAM_CS}: track 0.00 -> 57.9 mm
- net /VA12: track 0.00 -> 49.3 mm
- net /VA0: track 0.00 -> 46.5 mm, vias 0 -> 1
- net /BD7: track 0.00 -> 45.2 mm, vias 0 -> 1
- net /~{BLK2}: track 0.00 -> 45.1 mm
- net /~{BLK3}: track 0.00 -> 43.7 mm
- net /~{BLK1}: track 0.00 -> 42.5 mm
- net /VA2: track 0.00 -> 41.3 mm, vias 0 -> 1
- net /BD6: track 0.00 -> 40.0 mm, vias 0 -> 1
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Other:
- board text added: "27-MAY-2026: Untested"
- board text removed: "26-MAY-2026: Work In Progress"
