File: Internal_40KB/KiCad/VIC-20_Internal_40KB_RAM.kicad_sch (KiCad schematic)
At the start: 18 parts, among them J1 BLK Decoder, J2 RAM Decoder, J3 Disable/Enable Switch, J4 UD4, J5 UE4, U1 74LS20, U2 74LS138, U3 74LS138, U4 74HCT30, U5 74LS157, U6 CY62128Exx-xxS

Commit message: Initial design completed
Parts:
- U6: value CY62128Exx-xxS -> 62128 SRAM
Other:
- note removed: "WORK IN PROGRESS"
- moved on the sheet: C1, C2, C3, C4, C5, C6, U1B, U1C, U4B, U6
