File: MFJ-1258/Kicad/MFJ-1258.kicad_sch (KiCad schematic)
At the start: 19 parts, among them J1 C64-UserPort, J2 Screw_Terminal_01x01, J3 Screw_Terminal_01x01, Q1 2N3906, Q2 2N3906, Q3 2N3906, U1 NE555P

Commit message: Re-layout/Re-draw PCB
A few years more experience using KiCad now, updated from KiCad 6 to KiCad 9
Parts:
- RV1, RV2: footprint Potentiometer_THT:Potentiometer_Runtron_RM-065_Vertical -> Potentiometer_THT:Potentiometer_Piher_PT-10-V10_Vertical
Other:
- company: www.youtube.com/@brfff -> Brett Hallen
