File: Internal_32KB/KiCad/VIC-20_Internal_32KB_RAM.kicad_sch (KiCad schematic)
At the start: 17 parts, among them J1 BLK Decoder, J2 RAM Decoder, J3 Disable/Enable Switch, J4 UD4, J5 UE4, U1 74HCT138, U2 74HCT138, U3 74HCT10, U4 74HCT30, U5 74HCT157, U6 62256

Commit message: Further design corrections
Parts:
- removed C4: 100nF, Capacitor_THT:C_Disc_D3.0mm_W2.0mm_P2.50mm, symbol Device:C
- removed C5: 200nF, Capacitor_THT:C_Disc_D3.0mm_W2.0mm_P2.50mm, symbol Device:C
- removed U2: 74HCT138, Package_DIP:DIP-16_W7.62mm, symbol 74xx:74HCT138
- removed U3: 74HCT10, Package_DIP:DIP-14_W7.62mm, symbol 74xx:74LS10
- removed U4: 74HCT30, Package_DIP:DIP-14_W7.62mm, symbol 74xx:74LS30
- removed U5: 74HCT157, Package_DIP:DIP-16_W7.62mm, symbol 74xx:74LS157
- added U1: ATF16V8, Package_DIP:DIP-20_W7.62mm, symbol Logic_Programmable:ATF16V8Bxx-xxPU
- renumbered J4 to J1, J5 to J2, J2 to J3, J1 to J4, J3 to J5, U1 to U2, U6 to U3
Connections:
- net ~{CS} is gone; now on net ~{RAM_CS}: U3.20 (~{CS})
- net ~{OE} is gone; now on net GND: U3.22 (~{OE})
- net +5V: now also J3.10 (Pin_10), J3.11 (Pin_11), J3.12 (Pin_12), J3.13 (Pin_13), J3.14 (Pin_14), J3.15 (Pin_15), J3.7 (Pin_7), J3.9 (Pin_9), U1.20 (V_{CC})
- net CA13: now also U1.2 (I1); no longer U3.26 (A13)
- net CA14: now also U1.4 (I3); no longer U3.1 (A14)
- net CA15: now also U1.5 (I4)
- net GND: now also J3.5 (Pin_5), J4.4 (Pin_4), J4.5 (Pin_5), U1.10 (GND)
- net VA0: now also J1.5 (Pin_5); no longer J2.5 (Pin_5)
- net VA1: now also J1.6 (Pin_6); no longer J2.6 (Pin_6)
- net VA2: now also J1.7 (Pin_7); no longer J2.7 (Pin_7)
- net VR/~{W}: now also J2.10 (Pin_10); no longer J1.10 (Pin_10)
- net ~{BLK1}: now also U1.6 (I5)
- net ~{BLK2}: now also U1.7 (I6)
- net ~{BLK3}: now also U1.8 (I7)
- net ~{BLK5}: now also U1.9 (I8); no longer J4.10 (Pin_10)
- net ~{RAM_CS}: now also U1.12 (I/O)
- net ENABLE: now reaches J5.2 (Pin_2), R1.2
- net ENABLE: now also U1.11 (I9)
- net SΦ2/G1 renamed SΦ2
- net SΦ2: now also U1.1 (I)
- net VA13/G1 renamed VA13
- net VA13: now also U1.3 (I2)
- net ~{BLK0}/~{G2A}: no longer names the net of J3.4 (Pin_4)
- net ~{BLK1_{OUT}} renamed ~{BLK1_OUT}
- net ~{BLK1_OUT}: now also U1.18 (I/O)
- net ~{BLK2_{OUT}} renamed ~{BLK2_OUT}
- net ~{BLK2_OUT}: now also U1.17 (I/O)
- net ~{BLK3_{OUT}} renamed ~{BLK3_OUT}
- net ~{BLK3_OUT}: now also U1.16 (I/O)
- new net RAM_A13: U1.13 (I/O), U3.26 (A13)
- new net RAM_A14: U1.14 (I/O), U3.1 (A14)
- new net ~{BLK5_OUT}: J4.10 (Pin_10), U1.15 (I/O)
- no-connect marks 25 -> 15
Other:
- note added: "Future: To support ~{BLK5} expansion we will need to add an additional 6264"
- note removed: "Add ~{BLK5} with additional 6264 in future?"
- note removed: "Read: ~{CS} low & VR/~{W} high → ~{OE} low Write: ~{CS} low & VR/~{W} low → ~{OE} high"
- moved on the sheet: C1, C2, C3, J1, J2, J3, J4, U2, U3
